Commit message: Science upgrades (#126)
* steppers seem to be working with this setup

* naming fixes

* updated launch file for jetson/base station

* OMFG ITS KINDA WORKING DOE

* added ranges for both scoops for independent tuning

* lmao

* current working iteration of science for comp

* cleaned up a bit

* more cleaning up

* addressed PR comments

---------

Co-authored-by: UMDLoop Jetson Orin NX <umdloop@gmail.com>
Co-authored-by: Adrian Cires <ciresadrian@hotmail.com>
Co-authored-by: duttaishan01 <duttaishan01@FIGARO.myguest.virtualbox.org>

File: src/description/ros2_control/science/science.dc.ros2_control.xacro (robot description, xacro)
@@ -11,4 +11,5 @@
         <param name="can_id">0x70</param>
       </hardware>
+<!--
       <joint name="dc_auger">
         <param name="node_id">0</param>
@@ -28,6 +29,6 @@
         <state_interface name="motor_temperature"/>
         <state_interface name="torque_current"/>
-      </joint>
-      <joint name="dc_scoop">
+      </joint> -->
+      <!-- <joint name="dc_scoop">
         <param name="node_id">1</param>
         <param name="joint_type">revolute</param>
@@ -46,5 +47,5 @@
         <state_interface name="motor_temperature"/>
         <state_interface name="torque_current"/>
-      </joint>
+      </joint> -->
     </ros2_control>
   </xacro:macro>

File: src/description/ros2_control/science/science.servo.ros2_control.xacro (robot description, xacro)
@@ -11,10 +11,10 @@
                 <param name="can_id">0x80</param>
             </hardware>
-            <joint name="servo_rack_and_pinion_l">
+            <joint name="servo_scoops_lift_f">
                 <param name="node_id">0x1</param>
                 <param name="gear_ratio">1</param>
-                <param name="max_pos">235</param> <!-- degrees -->
-                <param name ="meters_per_deg">0.00016666666</param> <!-- (TODO) convert motor position in degrees to displacement in meters -->
-                <param name="servo_type">standard</param> <!-- standard or continuous -->
+                <param name="max_vel">300</param> <!-- deg/s -->
+                <param name ="meters_per_deg">0.00016666666</param> <!-- (TODO) When prismatic, convert motor position in degrees to displacement in meters -->
+                <param name="servo_type">continuous</param> <!-- standard or continuous -->
                 <param name="joint_type">revolute</param> <!-- revolute or prismatic -->
                 <command_interface name="position"/>
@@ -29,10 +29,10 @@
                 <state_interface name="status"/>
             </joint>
-            <joint name="servo_rack_and_pinion_r">
-                <param name="node_id">0x2</param>
+            <joint name="servo_scoops_lift_b">
+                <param name="node_id">0x0</param>
                 <param name="gear_ratio">1</param>
-                <param name="max_pos">235</param> <!-- degrees -->
-                <param name ="meters_per_deg">0.00016666666</param> <!-- (TODO) convert motor position in degrees to displacement in meters -->
-                <param name="servo_type">standard</param> <!-- standard or continuous -->
+                <param name="max_vel">300</param> <!-- deg/s -->
+                <param name ="meters_per_deg">0.00016666666</param> <!-- (TODO) When prismatic, convert motor position in degrees to displacement in meters -->
+                <param name="servo_type">continuous</param> <!-- standard or continuous -->
                 <param name="joint_type">revolute</param> <!-- revolute or prismatic -->
                 <command_interface name="position"/>
@@ -47,6 +47,60 @@
                 <state_interface name="status"/>
             </joint>
-            <joint name="servo_scoop_a">
-                <param name="node_id">0x3</param> <!-- 0x5 -->
+            <joint name="servo_sampler_lift_f">
+                <param name="node_id">0x2</param>
+                <param name="gear_ratio">1</param>
+                <param name="max_vel">300</param> <!-- deg/s -->
+                <param name ="meters_per_deg">0.00016666666</param> <!-- (TODO) When prismatic, convert motor position in degrees to displacement in meters -->
+                <param name="servo_type">continuous</param> <!-- standard or continuous -->
+                <param name="joint_type">revolute</param> <!-- revolute or prismatic -->
+                <command_interface name="position"/>
+                <command_interface name="velocity"/>
+                <command_interface name="status_request"/>
+                <command_interface name="maintenance_request"/>
+                <command_interface name="maintenance_frame_high"/>
+                <command_interface name="maintenance_frame_low"/>
+                <command_interface name="maintenance_data_count"/>
+                <state_interface name="position"/>
+                <state_interface name="velocity"/>
+                <state_interface name="status"/>
+            </joint>
+            <joint name="servo_sampler_lift_b">
+                <param name="node_id">0x3</param>
+                <param name="gear_ratio">1</param>
+                <param name="max_vel">300</param> <!-- deg/s -->
+                <param name ="meters_per_deg">0.00016666666</param> <!-- (TODO) When prismatic, convert motor position in degrees to displacement in meters -->
+                <param name="servo_type">continuous</param> <!-- standard or continuous -->
+                <param name="joint_type">revolute</param> <!-- revolute or prismatic -->
+                <command_interface name="position"/>
+                <command_interface name="velocity"/>
+                <command_interface name="status_request"/>
+                <command_interface name="maintenance_request"/>
+                <command_interface name="maintenance_frame_high"/>
+                <command_interface name="maintenance_frame_low"/>
+                <command_interface name="maintenance_data_count"/>
+                <state_interface name="position"/>
+                <state_interface name="velocity"/>
+                <state_interface name="status"/>
+            </joint>
+            <joint name="servo_conveyor_belt">
+                <param name="node_id">0x4</param>
+                <param name="gear_ratio">1</param>
+                <param name="max_vel">300</param> <!-- deg/s -->
+                <param name ="meters_per_deg">0.00016666666</param> <!-- (TODO) When prismatic, convert motor position in degrees to displacement in meters -->
+                <param name="servo_type">continuous</param> <!-- standard or continuous -->
+                <param name="joint_type">revolute</param> <!-- revolute or prismatic -->
+                <command_interface name="position"/>
+                <command_interface name="velocity"/>
+                <command_interface name="status_request"/>
+                <command_interface name="maintenance_request"/>
+                <command_interface name="maintenance_frame_high"/>
+                <command_interface name="maintenance_frame_low"/>
+                <command_interface name="maintenance_data_count"/>
+                <state_interface name="position"/>
+                <state_interface name="velocity"/>
+                <state_interface name="status"/>
+            </joint>
+            <joint name="servo_scoop_f">
+                <param name="node_id">0x5</param> <!-- 0x5 -->
                 <param name="gear_ratio">1</param>
                 <param name="max_pos">178</param> <!-- degrees -->
@@ -65,5 +119,5 @@
             </joint>
             <joint name="servo_scoop_b">
-                <param name="node_id">0x5</param> <!-- 0x3 -->
+                <param name="node_id">0x6</param> <!-- 0x3 -->
                 <param name="gear_ratio">1</param>
                 <param name="max_pos">178</param> <!-- degrees -->
@@ -81,42 +135,6 @@
                 <state_interface name="status"/>
             </joint>
-            <joint name="servo_sampler_lift_l">
-                <param name="node_id">0x6</param>
-                <param name="gear_ratio">1</param>
-                <param name="max_pos">360</param> <!-- degrees -->
-                <param name ="meters_per_deg">0.00016666666</param> <!-- (TODO) convert motor position in degrees to displacement in meters -->
-                <param name="servo_type">standard</param> <!-- standard / continuous -->
-                <param name="joint_type">revolute</param> <!-- revolute / prismatic -->
-                <command_interface name="position"/>
-                <command_interface name="velocity"/>
-                <command_interface name="status_request"/>
-                <command_interface name="maintenance_request"/>
-                <command_interface name="maintenance_frame_high"/>
-                <command_interface name="maintenance_frame_low"/>
-                <command_interface name="maintenance_data_count"/>
-                <state_interface name="position"/>
-                <state_interface name="velocity"/>
-                <state_interface name="status"/>
-            </joint>
-            <joint name="servo_sampler_lift_r">
-                <param name="node_id">0x4</param>
-                <param name="gear_ratio">1</param>
-                <param name="max_pos">360</param> <!-- degrees -->
-                <param name ="meters_per_deg">0.00016666666</param> <!-- (TODO) convert motor position in degrees to displacement in meters -->
-                <param name="servo_type">standard</param> <!-- standard / continuous -->
-                <param name="joint_type">revolute</param> <!-- revolute / prismatic -->
-                <command_interface name="position"/>
-                <command_interface name="velocity"/>
-                <command_interface name="status_request"/>
-                <command_interface name="maintenance_request"/>
-                <command_interface name="maintenance_frame_high"/>
-                <command_interface name="maintenance_frame_low"/>
-                <command_interface name="maintenance_data_count"/>
-                <state_interface name="position"/>
-                <state_interface name="velocity"/>
-                <state_interface name="status"/>
-            </joint>
             <joint name="servo_auger_lift">
-                <param name="node_id">0x0</param>
+                <param name="node_id">0x7</param>
                 <param name="gear_ratio">1</param>
                 <param name="max_pos">270</param> <!-- degrees -->

File: src/description/ros2_control/science/science.talon.ros2_control.xacro (robot description, xacro)
@@ -16,6 +16,6 @@
         </xacro:unless>
       </hardware>
-      <joint name="talon_auger">
-        <param name="node_id">2</param>
+      <joint name="dc_auger">
+        <param name="node_id">5</param>
         <param name="joint_type">revolute</param>
         <!-- Motor config (goBilda Saturn 5303 Series 360 RPM) -->
@@ -37,6 +37,6 @@
         <state_interface name="status"/>
       </joint>
-      <joint name="talon_scoop">
-        <param name="node_id">0</param>
+      <joint name="dc_scoop">
+        <param name="node_id">6</param>
         <param name="joint_type">revolute</param>
         <!-- Motor config (Pololu 37D defaults) -->

File: src/description/urdf/athena_science.urdf.xacro (robot description, xacro)
@@ -27,7 +27,7 @@
     <xacro:servo_ros2_control name="servo" can_interface="$(arg can_interface)"/>
     <!-- Import dc ros2_control description -->
-    <xacro:dc_ros2_control name="dc" can_interface="$(arg can_interface)"/>
+    <!-- <xacro:dc_ros2_control name="dc" can_interface="$(arg can_interface)"/> -->
     <!-- Import talon ros2_control description -->
-    <!-- <xacro:talon_ros2_control name="talon" deactivate_talon="$(arg deactivate_talon)" can_interface="$(arg can_interface)"/> -->
+    <xacro:talon_ros2_control name="talon" deactivate_talon="$(arg deactivate_talon)" can_interface="$(arg can_interface)"/>
     <!-- Import laser ros2_control description (CAN-based) -->
     <xacro:laser_ros2_control name="spectrometry_laser" can_interface="$(arg can_interface)"/>
