Commit message: fixing up the required HWIs

File: src/description/ros2_control/science/science.laser.ros2_control.xacro (robot description, xacro)
@@ -6,5 +6,5 @@
                 <plugin>laser_ros2_control/LaserHardwareInterface</plugin>
                 <param name="can_interface">${can_interface}</param>
-                <param name="can_id">0x130</param>
+                <param name="can_id">0x100</param>
                 <param name="update_rate">10</param> <!-- Hz -->
                 <param name="logger_rate">5</param> <!-- Hz -->
@@ -12,4 +12,5 @@
             </hardware>
             <gpio name="${name}">
+                <param name="node_id">1</param>
                 <state_interface name="laser_state"/>
                 <state_interface name="temperature"/>

File: src/description/ros2_control/science/science.photodiode.ros2_control.xacro (robot description, xacro)
@@ -1,8 +1,8 @@
 <?xml version="1.0"?>
 <robot xmlns:xacro="http://www.ros.org/wiki/xacro">
-    <xacro:macro name="sensor_diode_ros2_control" params="name can_interface:=can0">
+    <xacro:macro name="photodiode_ros2_control" params="name can_interface:=can0">
         <ros2_control name="${name}" type="system">
             <hardware>
-                <plugin>sensor_diode_ros2_control/SensorDiodeHardwareInterface</plugin>
+                <plugin>photodiode_ros2_control/PhotodiodeHardwareInterface</plugin>
                 <param name="can_interface">${can_interface}</param>
                 <param name="can_id">0x110</param>
@@ -12,5 +12,6 @@
             </hardware>
             <gpio name="${name}">
-                <command_interface name="request_measurement"/>
+                <param name="node_id">0</param>
+                <command_interface name="request_measurement_rate"/>
                 <command_interface name="status_request"/>
                 <command_interface name="maintenance_request"/>

File: src/description/urdf/athena_science.urdf.xacro (robot description, xacro)
@@ -12,5 +12,5 @@
   <xacro:include filename="$(find description)/ros2_control/science/science.laser.ros2_control.xacro"/>
   <xacro:include filename="$(find description)/ros2_control/science/science.ccd.ros2_control.xacro"/>
-  <xacro:include filename="$(find description)/ros2_control/science/science.sensor_diode.ros2_control.xacro"/>
+  <xacro:include filename="$(find description)/ros2_control/science/science.photodiode.ros2_control.xacro"/>
   <xacro:include filename="$(find description)/ros2_control/science/science.led.ros2_control.xacro"/>
   <xacro:include filename="$(find description)/ros2_control/science/science.limit_switch.ros2_control.xacro"/>
@@ -36,6 +36,6 @@
     <!-- Import CCD ros2_control description (CAN-based) -->
     <xacro:ccd_ros2_control name="spectrometry_ccd" can_interface="$(arg can_interface)"/>
-    <!-- Import sensor diode ros2_control description (CAN-based) -->
-    <xacro:sensor_diode_ros2_control name="sensor_diode" can_interface="$(arg can_interface)"/>
+    <!-- Import photodiode ros2_control description (CAN-based) -->
+    <xacro:photodiode_ros2_control name="photodiode" can_interface="$(arg can_interface)"/>
     <!-- Import LED and limit switch ros2_control descriptions -->
     <xacro:science_led_ros2_control name="fluoro_led_hwi" can_interface="$(arg can_interface)"/>
