Commit message: working zed servo controller

File: src/description/ros2_control/drive/drive.servo.ros2_control.xacro (robot description, xacro)
@@ -1,5 +1,5 @@
 <?xml version="1.0"?>
 <robot xmlns:xacro="http://www.ros.org/wiki/xacro">
-    <xacro:macro name="servo_ros2_control" params="name">
+    <xacro:macro name="servo_ros2_control" params="name can_interface:=can0">
         <ros2_control name="${name}" type="system">
             <hardware>
@@ -7,12 +7,12 @@
                 <param name="update_rate">20</param> <!-- Hz -->
                 <param name="logger_rate">5</param> <!-- Hz -->
-                <param name="logger_state">1</param> <!-- 0 for off, 1 for on -->
-                <param name="can_interface">can0</param>
-                <param name="can_id">0x80</param>
+                <param name="logger_state">0</param> <!-- 0 for off, 1 for on -->
+                <param name="can_interface">${can_interface}</param>
+                <param name="can_id">0x140</param>
             </hardware>
             <joint name="zed_servo_joint">
                 <param name="node_id">0x1</param>
                 <param name="gear_ratio">1</param>
-                <param name="max_pos">235</param> <!-- degrees -->
+                <param name="max_pos">270</param> <!-- degrees -->
                 <param name ="meters_per_deg">0.00016666666</param> <!-- (TODO) convert motor position in degrees to displacement in meters -->
                 <param name="servo_type">standard</param> <!-- standard or continuous -->

File: src/description/urdf/athena_drive.urdf.xacro (robot description, xacro)
@@ -65,5 +65,5 @@
     <xacro:power_module_ros2_control name="drive_power_module" can_interface="$(arg can_interface)"/>
     <!-- Servo control for Zed camera -->
-    <xacro:servo_ros2_control name="zed_servo_control"/>
+    <xacro:servo_ros2_control name="zed_servo_control" can_interface="$(arg can_interface)"/>
   </xacro:unless>
 </robot>
