Commit message: reorganizing files, fixing files to allow for colcon build --symlink-install, modified files for more improved launch setup

File: src/description/ros2_control/drive/drive.odrive.ros2_control.xacro (robot description, xacro)
@@ -1,5 +1,5 @@
 <?xml version="1.0"?>
 <robot xmlns:xacro="http://www.ros.org/wiki/xacro">
-  <xacro:macro name="odrive_ros2_control" params="name deactivate_odrive can_interface:=can0">
+  <xacro:macro name="odrive_ros2_control" params="name deactivate_odrive steering_config:=rear can_interface:=can0">
     <ros2_control name="${name}" type="system">
       <hardware>
@@ -16,30 +16,60 @@
         </xacro:unless>
       </hardware>
-      <joint name="steer_bl_joint">
-        <param name="node_id">7</param>
-        <param name="gear_ratio">26</param>
-        <command_interface name="position"/>
-        <command_interface name="velocity"/>
-        <!-- <command_interface name="status_request"/>
-        <command_interface name="maintenance_request"/> -->
-        <state_interface name="position"/>
-        <state_interface name="velocity"/>
-        <state_interface name="motor_temperature"/>
-        <state_interface name="torque_current"/>
-        <!-- <state_interface name="status"/> -->
-      </joint>
-      <joint name="steer_br_joint">
-        <param name="node_id">5</param>
-        <param name="gear_ratio">26</param>
-        <command_interface name="position"/>
-        <command_interface name="velocity"/>
-        <!-- <command_interface name="status_request"/>
-        <command_interface name="maintenance_request"/> -->
-        <state_interface name="position"/>
-        <state_interface name="velocity"/>
-        <state_interface name="motor_temperature"/>
-        <state_interface name="torque_current"/>
-        <!-- <state_interface name="status"/> -->
-      </joint>
+      <xacro:if value="${steering_config == 'front' or steering_config == 'all'}">
+        <joint name="steer_fl_joint">
+          <param name="node_id">6</param>
+          <param name="gear_ratio">26</param>
+          <command_interface name="position"/>
+          <command_interface name="velocity"/>
+          <!-- <command_interface name="status_request"/>
+          <command_interface name="maintenance_request"/> -->
+          <state_interface name="position"/>
+          <state_interface name="velocity"/>
+          <state_interface name="motor_temperature"/>
+          <state_interface name="torque_current"/>
+          <!-- <state_interface name="status"/> -->
+        </joint>
+        <joint name="steer_fr_joint">
+          <param name="node_id">4</param>
+          <param name="gear_ratio">26</param>
+          <command_interface name="position"/>
+          <command_interface name="velocity"/>
+          <!-- <command_interface name="status_request"/>
+          <command_interface name="maintenance_request"/> -->
+          <state_interface name="position"/>
+          <state_interface name="velocity"/>
+          <state_interface name="motor_temperature"/>
+          <state_interface name="torque_current"/>
+          <!-- <state_interface name="status"/> -->
+        </joint>
+      </xacro:if>
+      <xacro:if value="${steering_config == 'rear' or steering_config == 'all'}">
+        <joint name="steer_bl_joint">
+          <param name="node_id">7</param>
+          <param name="gear_ratio">26</param>
+          <command_interface name="position"/>
+          <command_interface name="velocity"/>
+          <!-- <command_interface name="status_request"/>
+          <command_interface name="maintenance_request"/> -->
+          <state_interface name="position"/>
+          <state_interface name="velocity"/>
+          <state_interface name="motor_temperature"/>
+          <state_interface name="torque_current"/>
+          <!-- <state_interface name="status"/> -->
+        </joint>
+        <joint name="steer_br_joint">
+          <param name="node_id">5</param>
+          <param name="gear_ratio">26</param>
+          <command_interface name="position"/>
+          <command_interface name="velocity"/>
+          <!-- <command_interface name="status_request"/>
+          <command_interface name="maintenance_request"/> -->
+          <state_interface name="position"/>
+          <state_interface name="velocity"/>
+          <state_interface name="motor_temperature"/>
+          <state_interface name="torque_current"/>
+          <!-- <state_interface name="status"/> -->
+        </joint>
+      </xacro:if>
     </ros2_control>
   </xacro:macro>
