Commit message: should be good

File: src/description/ros2_control/arm/arm.smc_2dof.ros2_control.xacro (robot description, xacro)
@@ -28,9 +28,9 @@
         <state_interface name="status"/>
       </joint>
-      <joint name="wrist_pitch">
+      <!-- <joint name="wrist_pitch">
         <param name="node_id">0x147</param>
         <param name="gear_ratio">40</param>
         <param name="joint_orientation">1.0</param>
-        <param name="operating_velocity">1000</param> <!-- motor dps -->
+        <param name="operating_velocity">1000</param> <!- motor dps ->
         <command_interface name="position"/>
         <command_interface name="velocity"/>
@@ -45,5 +45,5 @@
         <state_interface name="torque_current"/>
         <state_interface name="status"/>
-      </joint>
+      </joint> -->
       <joint name="wrist_roll">
         <param name="node_id">0x145</param>

File: src/description/ros2_control/arm/arm.talon_2dof.ros2_control.xacro (robot description, xacro)
@@ -16,4 +16,25 @@
         </xacro:unless>
       </hardware>
+      <joint name="wrist_pitch">
+        <param name="node_id">0</param>
+        <param name="joint_type">revolute</param>
+        <!-- Motor config (Pololu 37D defaults) -->
+        <param name="encoder_resolution">64.0</param>
+        <param name="gear_ratio">102.08</param>
+        <param name="inverted">true</param>
+        <param name="sensor_phase">true</param>
+        <param name="kP">0.25</param>
+        <param name="kI">0.0</param>
+        <param name="kD">0.0</param>
+        <param name="kF">0.0</param>
+        <command_interface name="position"/>
+        <command_interface name="velocity"/>
+        <command_interface name="status_request"/>
+        <state_interface name="position"/>
+        <state_interface name="velocity"/>
+        <state_interface name="motor_temperature"/>
+        <state_interface name="torque_current"/>
+        <state_interface name="status"/>
+      </joint>
       <joint name="gripper_claw">
         <param name="node_id">4</param>
